File: Software/brd_inject_test/data/VW_PCB.brd (EAGLE design)
At the start: 1 part

Commit message: main feature implemented in brd_inject_test folder
Connections:
- net S$1: now also E$1.3V3, E$1.ROW10, E$1.ROW14, E$1.ROW16; no longer E$1.ROW1, E$1.ROW9
- net S$2: now also E$1.GND1, E$1.ROW1, E$1.ROW4, E$1.ROW6; no longer E$1.ROW10
