File: Software/VirtualWire_User_App/Sample_Schematic_File/Servo_Control.sch (EAGLE design)
At the start: 4 parts

Commit message: polishing, bug fixes, Examples added
Parts:
- added BT1: SL-150-1/2AA/PR, battery:SL-150-1/2AA/PR
- renumbered C1 to CP1, C2 to CP2, R1 to RP1
Connections:
- new net N$2: BT1.+, SV1.1
- net A5V: no longer SV1.3
- net GND1: now also BT1.-, SV1.3; no longer SV1.1
Changed lines of the file:
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@@
 </classes>
 <parts>
-<part name="C1" library="capacitor-wima" library_urn="urn:adsk.eagle:library:116" deviceset="C" device="2,5-3" package3d_urn="urn:adsk.eagle:package:5436/1"/>
-<part name="C2" library="capacitor-wima" library_urn="urn:adsk.eagle:library:116" deviceset="C" device="2,5-3" package3d_urn="urn:adsk.eagle:package:5436/1"/>
-<part name="R1" library="rcl" library_urn="urn:adsk.eagle:library:334" deviceset="R-TRIMM" device="4G/J" package3d_urn="urn:adsk.eagle:package:23728/1"/>
+<part name="CP1" library="capacitor-wima" library_urn="urn:adsk.eagle:library:116" deviceset="C" device="2,5-3" package3d_urn="urn:adsk.eagle:package:5436/1"/>
+<part name="CP2" library="capacitor-wima" library_urn="urn:adsk.eagle:library:116" deviceset="C" device="2,5-3" package3d_urn="urn:adsk.eagle:package:5436/1"/>
+<part name="RP1" library="rcl" library_urn="urn:adsk.eagle:library:334" deviceset="R-TRIMM" device="4G/J" package3d_urn="urn:adsk.eagle:package:23728/1"/>
 <part name="SV1" library="con-lstb" library_urn="urn:adsk.eagle:library:162" deviceset="MA03-1" device="" package3d_urn="urn:adsk.eagle:package:8339/1"/>
 <part name="P+1" library="supply1" library_urn="urn:adsk.eagle:library:371" deviceset="VCC" device=""/>
 <part name="GND1" library="supply1" library_urn="urn:adsk.eagle:library:371" deviceset="GND" device=""/>
+<part name="BT1" library="battery" library_urn="urn:adsk.eagle:library:109" deviceset="SL-150-1/2AA/PR" device="" package3d_urn="urn:adsk.eagle:package:4607/1"/>
 </parts>
 <sheets>
@@
 </plain>
 <instances>
-<instance part="C1" gate="G$1" x="48.26" y="53.34" smashed="yes">
+<instance part="CP1" gate="G$1" x="48.26" y="53.34" smashed="yes">
 <attribute name="NAME" x="49.784" y="53.721" size="1.778" layer="95"/>
 <attribute name="VALUE" x="49.784" y="48.641" size="1.778" layer="96"/>
 </instance>
-<instance part="C2" gate="G$1" x="96.52" y="53.34" smashed="yes">
+<instance part="CP2" gate="G$1" x="96.52" y="53.34" smashed="yes">
 <attribute name="NAME" x="98.044" y="53.721" size="1.778" layer="95"/>
 <attribute name="VALUE" x="98.044" y="48.641" size="1.778" layer="96"/>
 </instance>
-<instance part="R1" gate="G$1" x="58.42" y="53.34" smashed="yes">
+<instance part="RP1" gate="G$1" x="58.42" y="53.34" smashed="yes">
 <attribute name="NAME" x="52.451" y="49.53" size="1.778" layer="95" rot="R90"/>
 <attribute name="VALUE" x="54.61" y="49.53" size="1.778" layer="96" rot="R90"/>
@@
 <attribute name="VALUE" x="78.74" y="5.08" size="1.778" layer="96"/>
 </instance>
+<instance part="BT1" gate="G$1" x="132.08" y="68.58"/>
 </instances>
 <busses>
@@
 <net name="A5V" class="0">
 <segment>
-<pinref part="C1" gate="G$1" pin="1"/>
+<pinref part="CP1" gate="G$1" pin="1"/>
 <wire x1="48.26" y1="55.88" x2="48.26" y2="60.96" width="0.1524" layer="91"/>
 <wire x1="48.26" y1="60.96" x2="45.72" y2="60.96" width="0.1524" layer="91"/>
-<pinref part="R1" gate="G$1" pin="E"/>
+<pinref part="RP1" gate="G$1" pin="E"/>
 <wire x1="48.26" y1="60.96" x2="58.42" y2="60.96" width="0.1524" layer="91"/>
 <wire x1="58.42" y1="60.96" x2="58.42" y2="58.42" width="0.1524" layer="91"/>
 <wire x1="45.72" y1="60.96" x2="45.72" y2="71.12" width="0.1524" layer="91"/>
 <wire x1="45.72" y1="71.12" x2="78.74" y2="71.12" width="0.1524" layer="91"/>
-<pinref part="C2" gate="G$1" pin="1"/>
+<pinref part="CP2" gate="G$1" pin="1"/>
 <wire x1="78.74" y1="71.12" x2="104.14" y2="71.12" width="0.1524" layer="91"/>
 <wire x1="96.52" y1="55.88" x2="96.52" y2="60.96" width="0.1524" layer="91"/>
 <wire x1="96.52" y1="60.96" x2="104.14" y2="60.96" width="0.1524" layer="91"/>
-<pinref part="SV1" gate="G$1" pin="3"/>
-<wire x1="104.14" y1="60.96" x2="116.84" y2="60.96" width="0.1524" layer="91"/>
-<wire x1="116.84" y1="60.96" x2="116.84" y2="53.34" width="0.1524" layer="91"/>
 <wire x1="104.14" y1="71.12" x2="104.14" y2="60.96" width="0.1524" layer="91"/>
-<junction x="104.14" y="60.96"/>
 <pinref part="P+1" gate="VCC" pin="VCC"/>
 <wire x1="78.74" y1="81.28" x2="78.74" y2="71.12" width="0.1524" layer="91"/>
@@
 <net name="GND1" class="0">
 <segment>
-<pinref part="R1" gate="G$1" pin="A"/>
+<pinref part="RP1" gate="G$1" pin="A"/>
 <wire x1="58.42" y1="48.26" x2="58.42" y2="43.18" width="0.1524" layer="91"/>
 <wire x1="58.42" y1="43.18" x2="53.34" y2="43.18" width="0.1524" layer="91"/>
-<pinref part="C1" gate="G$1" pin="2"/>
+<pinref part="CP1" gate="G$1" pin="2"/>
 <wire x1="53.34" y1="43.18" x2="48.26" y2="43.18" width="0.1524" layer="91"/>
 <wire x1="48.26" y1="43.18" x2="48.26" y2="48.26" width="0.1524" layer="91"/>
 <wire x1="53.34" y1="43.18" x2="53.34" y2="22.86" width="0.1524" layer="91"/>
 <junction x="53.34" y="43.18"/>
-<pinref part="SV1" gate="G$1" pin="1"/>
-<wire x1="116.84" y1="48.26" x2="116.84" y2="40.64" width="0.1524" layer="91"/>
-<wire x1="116.84" y1="40.64" x2="106.68" y2="40.64" width="0.1524" layer="91"/>
-<pinref part="C2" gate="G$1" pin="2"/>
+<pinref part="CP2" gate="G$1" pin="2"/>
 <wire x1="106.68" y1="40.64" x2="96.52" y2="40.64" width="0.1524" layer="91"/>
 <wire x1="96.52" y1="40.64" x2="96.52" y2="48.26" width="0.1524" layer="91"/>
@@
 <wire x1="81.28" y1="22.86" x2="106.68" y2="22.86" width="0.1524" layer="91"/>
 <wire x1="106.68" y1="22.86" x2="106.68" y2="40.64" width="0.1524" layer="91"/>
-<junction x="106.68" y="40.64"/>
 <pinref part="GND1" gate="1" pin="GND"/>
 <wire x1="81.28" y1="22.86" x2="81.28" y2="10.16" width="0.1524" layer="91"/>
 <junction x="81.28" y="22.86"/>
+<pinref part="SV1" gate="G$1" pin="3"/>
+<pinref part="BT1" gate="G$1" pin="-"/>
+<wire x1="116.84" y1="53.34" x2="127" y2="53.34" width="0.1524" layer="91"/>
+<wire x1="127" y1="53.34" x2="127" y2="68.58" width="0.1524" layer="91"/>
+<wire x1="116.84" y1="53.34" x2="106.68" y2="53.34" width="0.1524" layer="91"/>
+<wire x1="106.68" y1="53.34" x2="106.68" y2="40.64" width="0.1524" layer="91"/>
+<junction x="116.84" y="53.34"/>
+<junction x="106.68" y="40.64"/>
 </segment>
 </net>
@@
 <net name="A0" class="0">
 <segment>
-<pinref part="R1" gate="G$1" pin="S"/>
+<pinref part="RP1" gate="G$1" pin="S"/>
 <wire x1="63.5" y1="53.34" x2="63.5" y2="48.26" width="0.1524" layer="91"/>
 <label x="63.5" y="43.18" size="1.778" layer="95"/>
 </segment>
 </net>
+<net name="N$2" class="0">
+<segment>
+<pinref part="BT1" gate="G$1" pin="+"/>
+<pinref part="SV1" gate="G$1" pin="1"/>
+<wire x1="137.16" y1="68.58" x2="137.16" y2="48.26" width="0.1524" layer="91"/>
+<wire x1="137.16" y1="48.26" x2="116.84" y2="48.26" width="0.1524" layer="91"/>
+</segment>
+</net>
