File: Software/VirtualWire_User_App/VW_Eagle/data/PCB/VW_PCB.brd (EAGLE design)
At the start: 1 part

Commit message: eagle app visualizer polishing
Connections:
- new net S$1: E$1.5V, E$1.ROW1
- new net S$2: E$1.GND1, E$1.ROW3
- new net S$3: E$1.A0, E$1.ROW16
- new net S$4: E$1.D9, E$1.ROW15

Commit message: visualize wires in eagle app
Connections:
- net S$1: now also E$1.GND1, E$1.ROW2, E$1.ROW3; no longer E$1.5V, E$1.ROW1
- net S$2: now also E$1.5V, E$1.ROW16; no longer E$1.GND1, E$1.ROW3
- net S$3: now also E$1.ROW7; no longer E$1.ROW16
- net S$4: now also E$1.ROW10; no longer E$1.ROW15
Changed lines of the file:
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@@
       <signals>
         <signal name="S$1">
-          <contactref element="E$1" pad="5V"/>
-          <contactref element="E$1" pad="ROW1"/>
-          <wire extent="1-16" layer="19" width="0" x1="38.1" x2="17.78" y1="2.54" y2="35.306"/>
+          <contactref element="E$1" pad="ROW3"/>
+          <contactref element="E$1" pad="ROW2"/>
+          <wire extent="1-16" layer="19" width="0" x1="17.78" x2="17.78" y1="30.226" y2="32.766"/>
+          <contactref element="E$1" pad="GND1"/>
+          <wire extent="1-16" layer="19" width="0" x1="17.78" x2="40.64" y1="32.766" y2="2.54"/>
         </signal>
         <signal name="S$2">
-          <contactref element="E$1" pad="GND1"/>
-          <contactref element="E$1" pad="ROW3"/>
-          <wire extent="1-16" layer="19" width="0" x1="40.64" x2="17.78" y1="2.54" y2="30.226"/>
+          <contactref element="E$1" pad="5V"/>
+          <contactref element="E$1" pad="ROW16"/>
+          <wire extent="1-16" layer="19" width="0" x1="38.1" x2="54.61" y1="2.54" y2="17.526"/>
         </signal>
         <signal name="S$3">
           <contactref element="E$1" pad="A0"/>
-          <contactref element="E$1" pad="ROW16"/>
-          <wire extent="1-16" layer="19" width="0" x1="50.8" x2="54.61" y1="2.54" y2="17.526"/>
+          <contactref element="E$1" pad="ROW7"/>
+          <wire extent="1-16" layer="19" width="0" x1="50.8" x2="17.78" y1="2.54" y2="20.066"/>
         </signal>
         <signal name="S$4">
           <contactref element="E$1" pad="D9"/>
-          <contactref element="E$1" pad="ROW15"/>
-          <wire extent="1-16" layer="19" width="0" x1="39.116" x2="54.61" y1="50.8" y2="20.066"/>
+          <contactref element="E$1" pad="ROW10"/>
+          <wire extent="1-16" layer="19" width="0" x1="39.116" x2="54.61" y1="50.8" y2="32.766"/>
         </signal>
       </signals>
