File: Software/VirtualWire_User_App/VW_Fritzing/data/PCB/VW_PCB.brd (EAGLE design)
At the start: 1 part

Commit message: polishing, bug fixes, Examples added
Connections:
- new net S$1: E$1.GND1, E$1.ROW1, E$1.ROW3
- new net S$2: E$1.A5V, E$1.ROW11, E$1.ROW6
- new net S$3: E$1.ROW13, E$1.ROW4
- new net S$4: E$1.GND2, E$1.ROW16
- new net S$5: E$1.ROW10, E$1.ROW5
